File: DIY Arduino/Arduino/design_files/Arduino.kicad_pcb (KiCad board)
At the start: 2 copper layers, 68.6 x 53.3 mm, 45 parts, among them CON1 ISP, J1 USB_B, J2 BARREL_JACK, J3 PWR_SEL, P1 Power, P2 Analog, P3 Digital, P4 Digital, P5 CONN_01X01, P6 CONN_01X01, P7 CONN_01X01, P8 CONN_01X01, SW1 Reset, U1 LM7805, U2 FT231XS, U3 74LS125, U4 MCP1700T, U5 ATMEGA328P-PU, Y1 16Mhz

Commit message: Updates
Other:
- board text added: "DIY Ardu"
- board text added: "Rev 0.2 Aug 2020"
- board text removed: "DIY Arduino"
- board text removed: "DIY Arduino!"
- board text removed: "Rev 0.1 Oct 2018"
Changed lines of the file:
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@@
-(kicad_pcb (version 4) (host pcbnew 4.0.7)
+(kicad_pcb (version 4) (host pcbnew 4.0.6)
   (general
     (links 114)
@@
     (area 110.922999 72.949999 179.653001 126.440001)
     (thickness 1.6)
-    (drawings 50)
+    (drawings 52)
     (tracks 762)
     (zones 0)
@@
     (visible_elements 7FFFFFFF)
     (pcbplotparams
-      (layerselection 0x00030_80000001)
+      (layerselection 0x010f0_80000001)
       (usegerberextensions false)
       (excludeedgelayer true)
@@
       (outputformat 1)
       (mirror false)
-      (drillshape 1)
+      (drillshape 0)
       (scaleselection 1)
-      (outputdirectory ""))
+      (outputdirectory gerbers/))
   )
   (net 0 "")
@@
     )
   )
+  (dimension 53.34 (width 0.3) (layer Dwgs.User)
+    (gr_text "53.340 mm" (at 101.774 99.695 270) (layer Dwgs.User)
+      (effects (font (size 1.5 1.5) (thickness 0.3)))
+    )
+    (feature1 (pts (xy 110.998 126.365) (xy 100.424 126.365)))
+    (feature2 (pts (xy 110.998 73.025) (xy 100.424 73.025)))
+    (crossbar (pts (xy 103.124 73.025) (xy 103.124 126.365)))
+    (arrow1a (pts (xy 103.124 126.365) (xy 102.537579 125.238496)))
+    (arrow1b (pts (xy 103.124 126.365) (xy 103.710421 125.238496)))
+    (arrow2a (pts (xy 103.124 73.025) (xy 102.537579 74.151504)))
+    (arrow2b (pts (xy 103.124 73.025) (xy 103.710421 74.151504)))
+  )
+  (dimension 68.58 (width 0.3) (layer Dwgs.User)
+    (gr_text "68.580 mm" (at 145.288 68.627) (layer Dwgs.User)
+      (effects (font (size 1.5 1.5) (thickness 0.3)))
+    )
+    (feature1 (pts (xy 179.578 73.025) (xy 179.578 67.277)))
+    (feature2 (pts (xy 110.998 73.025) (xy 110.998 67.277)))
+    (crossbar (pts (xy 110.998 69.977) (xy 179.578 69.977)))
+    (arrow1a (pts (xy 179.578 69.977) (xy 178.451496 70.563421)))
+    (arrow1b (pts (xy 179.578 69.977) (xy 178.451496 69.390579)))
+    (arrow2a (pts (xy 110.998 69.977) (xy 112.124504 70.563421)))
+    (arrow2b (pts (xy 110.998 69.977) (xy 112.124504 69.390579)))
+  )
   (gr_text Diode (at 130.683 120.269) (layer F.SilkS)
     (effects (font (size 1 1) (thickness 0.15)))
@@
     (effects (font (size 1.5 1.25) (thickness 0.3)) (justify right mirror))
   )
-  (gr_text "Rev 0.1\nOct 2018" (at 160.02 95.885) (layer B.SilkS)
+  (gr_text "Rev 0.2\nAug 2020" (at 160.02 95.885) (layer B.SilkS)
     (effects (font (size 1.5 1.5) (thickness 0.3)) (justify mirror))
   )
-  (gr_text "DIY Arduino" (at 158.75 85.09) (layer B.SilkS)
+  (gr_text "DIY Ardu" (at 158.75 85.09) (layer B.SilkS)
     (effects (font (size 3 3) (thickness 0.5)) (justify mirror))
   )
-  (gr_text "DIY Arduino!" (at 158.623 117.221) (layer F.SilkS)
+  (gr_text "DIY Ardu" (at 158.623 117.221) (layer F.SilkS)
     (effects (font (size 2.5 3) (thickness 0.625) italic))
   )
